Commit message: 2021 03 04

File: humic_description/urdf/humic.gazebo.xacro (robot description, xacro)
@@ -5,10 +5,10 @@
     <gazebo>
         <plugin name="gazebo_ros_control" filename="libgazebo_ros_control.so">
-            <robotNamespace>/humic</robotNamespace>
+            <robotNamespace>humic</robotNamespace>
             <robotSimType>gazebo_ros_control/DefaultRobotHWSim</robotSimType>
         </plugin>
     </gazebo>
     <!-- mobile platform controller plugin-->
-    <!-- <gazebo>
+    <gazebo>
         <plugin name="mecanum_steering" filename="libgazebo_ros_planar_move.so">
             <updateRate>100.0</updateRate>
@@ -28,5 +28,5 @@
             <broadcastTF>true</broadcastTF>
         </plugin>
-    </gazebo> -->
+    </gazebo>
     <!-- camera controller plugin-->
     <gazebo reference="camera_link">
@@ -79,5 +79,5 @@
         </sensor>
     </gazebo>
-    <!-- <gazebo reference="ultrasonic1">
+    <gazebo reference="front_ultrasound">
         <material>Gazebo/Red</material>
         <sensor type="ray" name="sonar">
@@ -102,5 +102,5 @@
             <range>
               <min>0.01</min>
-              <max>1.0</max>
+              <max>2.0</max>
               <resolution>0.01</resolution>
             </range>
@@ -110,6 +110,6 @@
             <alwaysOn>true</alwaysOn>
             <updateRate>5</updateRate>
-            <topicName>/humic/sonar_front</topicName>
-            <frameName>ultrasonic1</frameName>
+            <topicName>/humic/front_ultrasound</topicName>
+            <frameName>front_ultrasound</frameName>
             <fov>0.5</fov>
             <radiation>ultrasound</radiation>
@@ -117,5 +117,5 @@
         </sensor>
     </gazebo>
-    <gazebo reference="ultrasonic2">
+    <gazebo reference="left_ultrasound">
         <material>Gazebo/Red</material>
         <sensor type="ray" name="sonar">
@@ -140,5 +140,5 @@
             <range>
               <min>0.01</min>
-              <max>1.0</max>
+              <max>2.0</max>
               <resolution>0.01</resolution>
             </range>
@@ -148,6 +148,6 @@
             <alwaysOn>true</alwaysOn>
             <updateRate>5</updateRate>
-            <topicName>/humic/sonar_left</topicName>
-            <frameName>ultrasonic2</frameName>
+            <topicName>/humic/left_ultrasound</topicName>
+            <frameName>left_ultrasound</frameName>
             <fov>0.5</fov>
             <radiation>ultrasound</radiation>
@@ -155,5 +155,5 @@
         </sensor>
     </gazebo>
-    <gazebo reference="ultrasonic3">
+    <gazebo reference="right_ultrasound">
         <material>Gazebo/Red</material>
         <sensor type="ray" name="sonar">
@@ -178,5 +178,5 @@
             <range>
               <min>0.01</min>
-              <max>1.0</max>
+              <max>2.0</max>
               <resolution>0.01</resolution>
             </range>
@@ -186,6 +186,6 @@
             <alwaysOn>true</alwaysOn>
             <updateRate>5</updateRate>
-            <topicName>/humic/sonar_right</topicName>
-            <frameName>ultrasonic3</frameName>
+            <topicName>/humic/right_ultrasound</topicName>
+            <frameName>right_ultrasound</frameName>
             <fov>0.5</fov>
             <radiation>ultrasound</radiation>
@@ -193,5 +193,5 @@
         </sensor>
     </gazebo>
-    <gazebo reference="ultrasonic4">
+    <gazebo reference="rear_ultrasound">
         <material>Gazebo/Red</material>
         <sensor type="ray" name="sonar">
@@ -216,5 +216,5 @@
             <range>
               <min>0.01</min>
-              <max>1.0</max>
+              <max>2.0</max>
               <resolution>0.01</resolution>
             </range>
@@ -224,11 +224,11 @@
             <alwaysOn>true</alwaysOn>
             <updateRate>5</updateRate>
-            <topicName>/humic/sonar_back</topicName>
-            <frameName>ultrasonic4</frameName>
+            <topicName>/humic/rear_ultrasound</topicName>
+            <frameName>rear_ultrasound</frameName>
             <fov>0.5</fov>
             <radiation>ultrasound</radiation>
           </plugin>
         </sensor>
-    </gazebo> -->
+    </gazebo>
     <!-- Robot Link-->
     <!-- mobile platform body-->
@@ -239,57 +239,57 @@
     <!-- mobile platform wheel -->
     <gazebo reference="rear_right_wheel_link">
-        <!-- <mu1>0.2</mu1>
-        <mu2>0.2</mu2> -->
-        <selfCollide>true</selfCollide>
-        <material>Gazebo/white</material>
-        <!-- <kp>500000.0</kp>
+        <mu1>0.2</mu1>
+        <mu2>0.2</mu2>
+        <selfCollide>true</selfCollide>
+        <material>Gazebo/white</material>
+        <kp>500000.0</kp>
         <kd>10.0</kd>
         <minDepth>0.001</minDepth>
         <maxVel>0.1</maxVel>
-        <fdirl>1 0 0</fdirl> -->
+        <fdirl>1 0 0</fdirl>
     </gazebo>
     <gazebo reference="front_left_wheel_link">
-        <!-- <mu1>0.2</mu1>
-        <mu2>0.2</mu2> -->
-        <selfCollide>true</selfCollide>
-        <material>Gazebo/white</material>
-        <!-- <kp>500000.0</kp>
+        <mu1>0.2</mu1>
+        <mu2>0.2</mu2>
+        <selfCollide>true</selfCollide>
+        <material>Gazebo/white</material>
+        <kp>500000.0</kp>
         <kd>10.0</kd>
         <minDepth>0.001</minDepth>
         <maxVel>0.1</maxVel>
-        <fdirl>1 0 0</fdirl> -->
+        <fdirl>1 0 0</fdirl>
     </gazebo>
     <gazebo reference="front_right_wheel_link">
-        <!-- <mu1>0.2</mu1>
-        <mu2>0.2</mu2> -->
-        <selfCollide>true</selfCollide>
-        <material>Gazebo/white</material>
-        <!-- <kp>500000.0</kp>
+        <mu1>0.2</mu1>
+        <mu2>0.2</mu2>
+        <selfCollide>true</selfCollide>
+        <material>Gazebo/white</material>
+        <kp>500000.0</kp>
         <kd>10.0</kd>
         <minDepth>0.001</minDepth>
         <maxVel>0.1</maxVel>
-        <fdirl>1 0 0</fdirl> -->
+        <fdirl>1 0 0</fdirl>
     </gazebo>
     <gazebo reference="rear_left_wheel_link">
-        <!-- <mu1>0.2</mu1>
-        <mu2>0.2</mu2> -->
-        <selfCollide>true</selfCollide>
-        <material>Gazebo/white</material>
-        <!-- <kp>500000.0</kp>
+        <mu1>0.2</mu1>
+        <mu2>0.2</mu2>
+        <selfCollide>true</selfCollide>
+        <material>Gazebo/white</material>
+        <kp>500000.0</kp>
         <kd>10.0</kd>
         <minDepth>0.001</minDepth>
         <maxVel>0.1</maxVel>
-        <fdirl>1 0 0</fdirl> -->
+        <fdirl>1 0 0</fdirl>
     </gazebo>
     <!-- column -->
     <gazebo reference="base_column_link">
-        <!-- <mu1>0.2</mu1>
-        <mu2>0.2</mu2> -->
+        <mu1>0.2</mu1>
+        <mu2>0.2</mu2>
         <selfCollide>true</selfCollide>
         <material>Gazebo/white</material>
     </gazebo>
     <gazebo reference="inner_column_link">
-        <!-- <mu1>0.2</mu1>
-        <mu2>0.2</mu2> -->
+        <mu1>0.2</mu1>
+        <mu2>0.2</mu2>
         <selfCollide>true</selfCollide>
         <material>Gazebo/white</material>
@@ -297,6 +297,6 @@
     <!-- Torso -->
     <gazebo reference="torso_link">
-        <!-- <mu1>0.2</mu1>
-        <mu2>0.2</mu2> -->
+        <mu1>0.2</mu1>
+        <mu2>0.2</mu2>
         <selfCollide>true</selfCollide>
         <material>Gazebo/Grey</material>
@@ -304,18 +304,40 @@
     <!-- head -->
     <gazebo reference="neck_link">
-        <!-- <mu1>0.2</mu1>
-        <mu2>0.2</mu2> -->
-        <selfCollide>true</selfCollide>
-        <material>Gazebo/Grey</material>
-    </gazebo>
-    <gazebo reference="neck_head_link">
-        <!-- <mu1>0.2</mu1>
-        <mu2>0.2</mu2> -->
+        <!-- <sensor type="contact" name="humic_contact_sensor">
+            <update_rate>1000.0</update_rate>
+            <always_on>true</always_on>
+            <contact>
+                <collision>neck_link_collision</collision>
+            </contact>
+            <plugin name="neck_link_plugin" filename="libgazebo_ros_bumper.so">
+                <bumperTopicName>humic/gazebo_contact</bumperTopicName>
+                <frameName>neck_link</frameName>
+            </plugin>
+        </sensor> -->
+        <mu1>0.2</mu1>
+        <mu2>0.2</mu2>
+        <selfCollide>true</selfCollide>
+        <material>Gazebo/Grey</material>
+    </gazebo>
+    <gazebo reference="head_link">
+        <!-- <sensor type="contact" name="humic_contact_sensor">
+            <update_rate>1000.0</update_rate>
+            <always_on>true</always_on>
+            <contact>
+                <collision>head_link_collision</collision>
+            </contact>
+            <plugin name="head_link_plugin" filename="libgazebo_ros_bumper.so">
+                <bumperTopicName>humic/gazebo_contact</bumperTopicName>
+                <frameName>head_link</frameName>
+            </plugin>
+        </sensor> -->
+        <mu1>0.2</mu1>
+        <mu2>0.2</mu2>
         <selfCollide>true</selfCollide>
         <material>Gazebo/Grey</material>
     </gazebo>
     <gazebo reference="head_kinect_link">
-        <!-- <mu1>0.2</mu1>
-        <mu2>0.2</mu2> -->
+        <mu1>0.2</mu1>
+        <mu2>0.2</mu2>
         <selfCollide>true</selfCollide>
         <material>Gazebo/Grey</material>
@@ -350,4 +372,15 @@
     </gazebo>
     <gazebo reference="r_upperArm_link">
+        <!-- <sensor type="contact" name="humic_contact_sensor">
+            <update_rate>1000.0</update_rate>
+            <always_on>true</always_on>
+            <contact>
+                <collision>r_upperArm_link_collision</collision>
+            </contact>
+            <plugin name="r_upperArm_link_plugin" filename="libgazebo_ros_bumper.so">
+                <bumperTopicName>humic/gazebo_contact</bumperTopicName>
+                <frameName>r_upperArm_link</frameName>
+            </plugin>
+        </sensor> -->
         <mu1>0.2</mu1>
         <mu2>0.2</mu2>
@@ -436,6 +469,6 @@
             </plugin>
         </sensor>
-        <!-- <mu1>0.2</mu1>
-        <mu2>0.2</mu2> -->
+        <mu1>0.2</mu1>
+        <mu2>0.2</mu2>
         <selfCollide>true</selfCollide>
         <material>Gazebo/Grey</material>
@@ -604,4 +637,15 @@
     </gazebo>
     <gazebo reference="l_upperArm_link">
+        <!-- <sensor type="contact" name="humic_contact_sensor">
+            <update_rate>1000.0</update_rate>
+            <always_on>true</always_on>
+            <contact>
+                <collision>l_upperArm_link_collision</collision>
+            </contact>
+            <plugin name="l_upperArm_link_plugin" filename="libgazebo_ros_bumper.so">
+                <bumperTopicName>humic/gazebo_contact</bumperTopicName>
+                <frameName>l_upperArm_link</frameName>
+            </plugin>
+        </sensor> -->
         <mu1>0.2</mu1>
         <mu2>0.2</mu2>
@@ -610,4 +654,15 @@
     </gazebo>
     <gazebo reference="l_elbow_link">
+        <!-- <sensor type="contact" name="humic_contact_sensor">
+            <update_rate>1000.0</update_rate>
+            <always_on>true</always_on>
+            <contact>
+                <collision>l_elbow_link_collision</collision>
+            </contact>
+            <plugin name="l_elbow_link_plugin" filename="libgazebo_ros_bumper.so">
+                <bumperTopicName>humic/gazebo_contact</bumperTopicName>
+                <frameName>l_elbow_link</frameName>
+            </plugin>
+        </sensor> -->
         <mu1>0.2</mu1>
         <mu2>0.2</mu2>
@@ -616,4 +671,15 @@
     </gazebo>
     <gazebo reference="l_foreArm_link">
+        <!-- <sensor type="contact" name="humic_contact_sensor">
+            <update_rate>1000.0</update_rate>
+            <always_on>true</always_on>
+            <contact>
+                <collision>l_foreArm_link_collision</collision>
+            </contact>
+            <plugin name="l_foreArm_link_plugin" filename="libgazebo_ros_bumper.so">
+                <bumperTopicName>humic/gazebo_contact</bumperTopicName>
+                <frameName>l_foreArm_link</frameName>
+            </plugin>
+        </sensor> -->
         <mu1>0.2</mu1>
         <mu2>0.2</mu2>
@@ -622,4 +688,15 @@
     </gazebo>
     <gazebo reference="l_lowerArm_link">
+        <!-- <sensor type="contact" name="humic_contact_sensor">
+            <update_rate>1000.0</update_rate>
+            <always_on>true</always_on>
+            <contact>
+                <collision>l_lowerArm_link_collision</collision>
+            </contact>
+            <plugin name="l_lowerArm_link_plugin" filename="libgazebo_ros_bumper.so">
+                <bumperTopicName>humic/gazebo_contact</bumperTopicName>
+                <frameName>l_lowerArm_link</frameName>
+            </plugin>
+        </sensor> -->
         <mu1>0.2</mu1>
         <mu2>0.2</mu2>
@@ -628,4 +705,15 @@
     </gazebo>
     <gazebo reference="l_wrist_link">
+        <!-- <sensor type="contact" name="humic_contact_sensor">
+            <update_rate>1000.0</update_rate>
+            <always_on>true</always_on>
+            <contact>
+                <collision>l_wrist_link_collision</collision>
+            </contact>
+            <plugin name="l_wrist_link_plugin" filename="libgazebo_ros_bumper.so">
+                <bumperTopicName>humic/gazebo_contact</bumperTopicName>
+                <frameName>l_wrist_link</frameName>
+            </plugin>
+        </sensor> -->
         <mu1>0.2</mu1>
         <mu2>0.2</mu2>
@@ -643,4 +731,15 @@
     </gazebo>
     <gazebo reference="l_finger1_1_link">
+        <!-- <sensor type="contact" name="humic_contact_sensor">
+            <update_rate>1000.0</update_rate>
+            <always_on>true</always_on>
+            <contact>
+                <collision>l_finger1_1_link_collision</collision>
+            </contact>
+            <plugin name="l_finger1_1_link_plugin" filename="libgazebo_ros_bumper.so">
+                <bumperTopicName>humic/gazebo_contact</bumperTopicName>
+                <frameName>l_finger1_1_link</frameName>
+            </plugin>
+        </sensor> -->
         <mu1>0.2</mu1>
         <mu2>0.2</mu2>
@@ -649,4 +748,15 @@
     </gazebo>
     <gazebo reference="l_finger1_2_link">
+        <!-- <sensor type="contact" name="humic_contact_sensor">
+            <update_rate>1000.0</update_rate>
+            <always_on>true</always_on>
+            <contact>
+                <collision>l_finger1_2_link_collision</collision>
+            </contact>
+            <plugin name="l_finger1_2_link_plugin" filename="libgazebo_ros_bumper.so">
+                <bumperTopicName>humic/gazebo_contact</bumperTopicName>
+                <frameName>l_finger1_2_link</frameName>
+            </plugin>
+        </sensor> -->
         <mu1>0.2</mu1>
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