Commit message: 2021 03 04

File: humic_description/urdf/humic.urdf.xacro (robot description, xacro)
@@ -1,9 +1,10 @@
 <?xml version="1.0"?>
 <robot name="humic" xmlns:xacro="http://ros.org/wiki/xacro">
-    <!-- Import all Gazebo-customization elements, including Gazebo colors -->
+    <xacro:include filename="$(find humic_description)/urdf/materials.xacro"/>
     <xacro:include filename="$(find humic_description)/urdf/humic.gazebo.xacro"/>
-    <!-- Import Rviz colors -->
-    <xacro:include filename="$(find humic_description)/urdf/materials.xacro"/>
-    <xacro:include filename="$(find humic_description)/urdf/humic.transmission.xacro"/>
+    <xacro:include filename="$(find humic_description)/urdf/humic.right_transmission.xacro"/>
+    <xacro:include filename="$(find humic_description)/urdf/humic.left_transmission.xacro"/>
+    <xacro:include filename="$(find humic_description)/urdf/humic.head_transmission.xacro"/>
+    <xacro:include filename="$(find humic_description)/urdf/humic.column_transmission.xacro"/>
     <!-- base footprint -->
     <link name="base_footprint"/>
@@ -33,10 +34,10 @@
         </inertial>
     </link>
-    <!-- <joint name="ultrasonic1_joint" type="fixed">
+    <joint name="front_ultrasound_joint" type="fixed">
         <origin xyz="0.12 0 0.038" rpy="0 0 0"/>
         <parent link="base_link"/>
-        <child link="ultrasonic1"/>
-    </joint>
-    <link name="ultrasonic1">
+        <child link="front_ultrasound"/>
+    </joint>
+    <link name="front_ultrasound">
         <visual>
             <origin xyz="0 0 0" rpy="0 0 0"/>
@@ -44,13 +45,13 @@
                 <box size="0.002 0.002 0.002"/>
             </geometry>
-            <material name="Red"/>
-        </visual>
-    </link>
-    <joint name="ultrasonic2_joint" type="fixed">
+            <material name="red"/>
+        </visual>
+    </link>
+    <joint name="left_ultrasound_joint" type="fixed">
         <origin xyz="-0.004 0.063 0.038" rpy="0 0 1.57"/>
         <parent link="base_link"/>
-        <child link="ultrasonic2"/>
-    </joint>
-    <link name="ultrasonic2">
+        <child link="left_ultrasound"/>
+    </joint>
+    <link name="left_ultrasound">
         <visual>
             <origin xyz="0 0 0" rpy="0 0 0"/>
@@ -58,13 +59,13 @@
                 <box size="0.002 0.002 0.002"/>
             </geometry>
-            <material name="Red"/>
-        </visual>
-    </link>
-    <joint name="ultrasonic3_joint" type="fixed">
+            <material name="red"/>
+        </visual>
+    </link>
+    <joint name="right_ultrasound_joint" type="fixed">
         <origin xyz="-0.004 -0.063 0.038" rpy="0 0 -1.57"/>
         <parent link="base_link"/>
-        <child link="ultrasonic3"/>
-    </joint>
-    <link name="ultrasonic3">
+        <child link="right_ultrasound"/>
+    </joint>
+    <link name="right_ultrasound">
         <visual>
             <origin xyz="0 0 0" rpy="0 0 0"/>
@@ -72,13 +73,13 @@
                 <box size="0.002 0.002 0.002"/>
             </geometry>
-            <material name="Red"/>
-        </visual>
-    </link>
-    <joint name="ultrasonic4_joint" type="fixed">
+            <material name="red"/>
+        </visual>
+    </link>
+    <joint name="rear_ultrasound_joint" type="fixed">
         <origin xyz="-0.117 0 0.038" rpy="0 0 3.14"/>
         <parent link="base_link"/>
-        <child link="ultrasonic4"/>
-    </joint>
-    <link name="ultrasonic4">
+        <child link="rear_ultrasound"/>
+    </joint>
+    <link name="rear_ultrasound">
         <visual>
             <origin xyz="0 0 0" rpy="0 0 0"/>
@@ -86,12 +87,12 @@
                 <box size="0.002 0.002 0.002"/>
             </geometry>
-            <material name="Red"/>
-        </visual>
-    </link> -->
+            <material name="red"/>
+        </visual>
+    </link>
     <!-- Mobile-Platform Wheel -->
     <!-- front left & rear right couple-->
     <!-- front right & rear left couple-->
-    <joint name="rear_left_wheel_joint" type="fixed"> <!-- continuous -->
-        <!-- <axis xyz="0 -1 0" /> -->
+    <joint name="rear_left_wheel_joint" type="continuous">
+        <axis xyz="0 -1 0" />
         <origin xyz="-0.085 0.085 0" rpy="0 0 0"/>
         <parent link="base_link"/>
@@ -118,6 +119,6 @@
         </inertial>
     </link>
-    <joint name="rear_right_wheel_joint" type="fixed"> <!-- continuous -->
-        <!-- <axis xyz="0 1 0" /> -->
+    <joint name="rear_right_wheel_joint" type="continuous">
+        <axis xyz="0 1 0" />
         <origin xyz="-0.085 -0.085 0" rpy="0 0 0"/>
         <parent link="base_link"/>
@@ -144,6 +145,6 @@
         </inertial>
     </link>
-    <joint name="front_right_wheel_joint" type="fixed"> <!-- continuous -->
-        <!-- <axis xyz="0 1 0" /> -->
+    <joint name="front_right_wheel_joint" type="continuous">
+        <axis xyz="0 1 0" />
         <origin xyz="0.085 0.085 0" rpy="0 0 0"/>
         <parent link="base_link"/>
@@ -170,6 +171,6 @@
         </inertial>
     </link>
-    <joint name="front_left_wheel_joint" type="fixed"> <!-- continuous -->
-        <!-- <axis xyz="0 -1 0" /> -->
+    <joint name="front_left_wheel_joint" type="continuous">
+        <axis xyz="0 -1 0" />
         <origin xyz="0.085 -0.085 0" rpy="0 0 0"/>
         <parent link="base_link"/>
@@ -196,5 +197,5 @@
         </inertial>
     </link>
-    <!-- Column -->
+    <!-- Lift Column -->
     <joint name="base_column_joint" type="fixed">
         <origin xyz="0 0 0" rpy="0 0 0"/>
@@ -222,7 +223,7 @@
         </inertial>
     </link>
-    <joint name="inner_column_joint" type="fixed"> <!--prismatic-->
-        <!-- <axis xyz="0 0 1" /> -->
-        <!-- <limit velocity="1" effort="1" lower="0" upper="0.10" /> -->
+    <joint name="inner_column_joint" type="prismatic">
+        <axis xyz="0 0 1" />
+        <limit velocity="1" effort="1" lower="0" upper="0.10" />
         <origin xyz="0.05 0 0.05" rpy="0 0 0"/>
         <parent link="base_column_link"/>
@@ -258,12 +259,4 @@
             <material name="grey"/>
         </visual>
-        <!-- <collision>
-            <origin xyz="-0.016 0 0.275" rpy="0 0 0"/>
-            <geometry>
-                <mesh
-                    filename="package://humic_description/meshes/STL/torso.stl" scale="0.01 0.01 0.01"/>
-            </geometry>
-            <material name="grey"/>
-        </collision> -->
         <collision>
             <origin xyz="-0.003 0 0.23" rpy="0 0 0"/>
@@ -297,13 +290,13 @@
         </inertial>
     </link>
-    <joint name="neck_joint" type="fixed"> <!-- revolute -->
-        <!-- <axis xyz="0 0 1" /> -->
-        <!-- <limit velocity="6.5" effort="1000" lower="-0.7854" upper="0.7854" /> -->
-        <!-- <dynamics damping="0.7"/> -->
+    <joint name="neck_joint" type="revolute">
+        <axis xyz="0 0 1" />
+        <limit velocity="6.5" effort="1000" lower="-0.7854" upper="0.7854" />
+        <dynamics damping="0.7"/>
         <origin xyz="0.023 0 0.337" rpy="0 0 0"/>
         <parent link="neck_link"/>
-        <child link="neck_head_link"/>
-    </joint>
-    <link name="neck_head_link">
+        <child link="head_link"/>
+    </joint>
+    <link name="head_link">
         <visual>
             <origin xyz="-0.073 0 -0.338" rpy="0 0 0"/>
@@ -319,11 +312,10 @@
         </inertial>
     </link>
-    <joint name="neck_head_joint" type="fixed"> <!-- revolute -->
-        <!-- <axis xyz="0 -1 0" /> -->
-        <!-- <limit velocity="6.5" effort="1000" lower="-0.7854" upper="0.7854" /> -->
-        <!-- <dynamics damping="0.7"/> -->
-        <!-- <origin xyz="0 0 0.02" rpy="0 0 0"/>  -->
+    <joint name="head_joint" type="revolute">
+        <axis xyz="0 -1 0" />
+        <limit velocity="6.5" effort="1000" lower="-0.7854" upper="0.7854" />
+        <dynamics damping="0.7"/>
         <origin xyz="0 0 0.02" rpy="0 0.6 0"/>
-        <parent link="neck_head_link"/>
+        <parent link="head_link"/>
         <child link="head_kinect_link"/>
     </joint>
@@ -409,5 +401,5 @@
         <limit velocity="6.5" effort="1000" lower="-3.14" upper="3.14" />
         <dynamics damping="0.7"/>
-        <origin xyz="0.004 -0.123 0.27" rpy="0 -1.57 0"/> <!-- 0 -1.57 0 -->
+        <origin xyz="0.004 -0.123 0.27" rpy="0 -1.57 0"/>
         <parent link="r_shoulder_link"/>
         <child link="r_upperArm_link"/>
@@ -436,5 +428,5 @@
     <joint name="r_upperArm_joint" type="revolute">
         <axis xyz="1 0 0" />
-        <limit velocity="6.5" effort="1000" lower="-1.57" upper="1.57" />
+        <limit velocity="6.5" effort="1000" lower="-1.57" upper="0" />
         <dynamics damping="0.7"/>
         <origin xyz="0 -0.011 0" rpy="0 0 0"/>
@@ -465,5 +457,5 @@
     <joint name="r_elbow_joint" type="revolute">
         <axis xyz="1 0 0" />
-        <limit velocity="6.5" effort="1000" lower="-1.57" upper="1.57" />
+        <limit velocity="6.5" effort="1000" lower="0" upper="0.52" />
         <dynamics damping="0.7"/>
         <origin xyz="0 0.011 -0.105" rpy="0 0 0"/>
@@ -523,5 +515,5 @@
     <joint name="r_lowerArm_joint" type="revolute">
         <axis xyz="1 0 0" />
-        <limit velocity="6.5" effort="1000" lower="-1.57" upper="1.57" />
+        <limit velocity="13" effort="1000" lower="-1.57" upper="1.57" />
         <dynamics damping="0.7"/>
         <origin xyz="0 0 -0.012" rpy="0 0 0"/>
@@ -552,5 +544,5 @@
     <joint name="r_wrist_joint" type="revolute">
         <axis xyz="0 0 -1" />
-        <limit velocity="6.5" effort="1000" lower="-1.57" upper="1.57" />
+        <limit velocity="13" effort="1000" lower="-1.57" upper="1.57" />
         <dynamics damping="0.7"/>
         <origin xyz="0 0 -0.048" rpy="0 0 0"/>
@@ -592,6 +584,6 @@
     <joint name="r_finger1_1_joint" type="revolute">
         <axis xyz="1 0 0" />
-        <limit velocity="5" effort="1" lower="0" upper="1.57" />
-        <dynamics damping="0.7"/>
+        <limit velocity="1" effort="1" lower="0" upper="1.57" />
+        <dynamics damping="0.2"/>
         <origin xyz="0.012 -0.006 -0.036" rpy="0 0 0"/>
         <parent link="r_finger_link"/>
@@ -621,6 +613,6 @@
     <joint name="r_finger1_2_joint" type="revolute">
         <axis xyz="1 0 0" />
-        <limit velocity="5" effort="1" lower="0" upper="1.57" />
-        <dynamics damping="0.7"/>
+        <limit velocity="1" effort="1" lower="0" upper="1.57" />
+        <dynamics damping="0.2"/>
         <origin xyz="0 0 -0.02" rpy="0 0 0"/>
         <parent link="r_finger1_1_link"/>
@@ -650,6 +642,6 @@
     <joint name="r_finger2_1_joint" type="revolute">
         <axis xyz="1 0 0" />
-        <limit velocity="5" effort="1" lower="0" upper="1.57" />
-        <dynamics damping="0.7"/>
+        <limit velocity="1" effort="1" lower="0" upper="1.57" />
+        <dynamics damping="0.2"/>
         <origin xyz="0.004 -0.006 -0.036" rpy="0 0 0"/>
         <parent link="r_finger_link"/>
@@ -679,6 +671,6 @@
     <joint name="r_finger2_2_joint" type="revolute">
         <axis xyz="1 0 0" />
-        <limit velocity="5" effort="1" lower="0" upper="1.57" />
-        <dynamics damping="0.7"/>
+        <limit velocity="1" effort="1" lower="0" upper="1.57" />
+        <dynamics damping="0.2"/>
         <origin xyz="0 0 -0.021" rpy="0 0 0"/>
         <parent link="r_finger2_1_link"/>
@@ -708,6 +700,6 @@
     <joint name="r_finger3_1_joint" type="revolute">
         <axis xyz="1 0 0" />
-        <limit velocity="5" effort="1" lower="0" upper="1.57" />
-        <dynamics damping="0.7"/>
+        <limit velocity="1" effort="1" lower="0" upper="1.57" />
+        <dynamics damping="0.2"/>
         <origin xyz="-0.004 -0.006 -0.036" rpy="0 0 0"/>
         <parent link="r_finger_link"/>
@@ -737,6 +729,6 @@
     <joint name="r_finger3_2_joint" type="revolute">
         <axis xyz="1 0 0" />
-        <limit velocity="5" effort="1" lower="0" upper="1.57" />
-        <dynamics damping="0.7"/>
+        <limit velocity="1" effort="1" lower="0" upper="1.57" />
+        <dynamics damping="0.2"/>
         <origin xyz="0 0 -0.017" rpy="0 0 0"/>
         <parent link="r_finger3_1_link"/>
@@ -766,6 +758,6 @@
     <joint name="r_finger4_1_joint" type="revolute">
         <axis xyz="1 0 0" />
-        <limit velocity="5" effort="1" lower="0" upper="1.57" />
-        <dynamics damping="0.7"/>
+        <limit velocity="1" effort="1" lower="0" upper="1.57" />
+        <dynamics damping="0.2"/>
         <origin xyz="-0.012 -0.006 -0.036" rpy="0 0 0"/>
         <parent link="r_finger_link"/>
@@ -795,6 +787,6 @@
     <joint name="r_finger4_2_joint" type="revolute">
         <axis xyz="1 0 0" />
-        <limit velocity="5" effort="1" lower="0" upper="1.57" />
-        <dynamics damping="0.7"/>
+        <limit velocity="1" effort="1" lower="0" upper="1.57" />
+        <dynamics damping="0.2"/>
         <origin xyz="0 0 -0.015" rpy="0 0 0"/>
         <parent link="r_finger4_1_link"/>
@@ -823,7 +815,7 @@
     </link>
     <joint name="r_thumb_joint" type="revolute">
-        <axis xyz="0 0 -1" />
-        <limit velocity="5" effort="1" lower="0" upper="0.785" />
-        <dynamics damping="0.7"/>
+        <axis xyz="0 0 1" />
+        <limit velocity="1" effort="1" lower="0" upper="0.785" />
+        <dynamics damping="0.2"/>
         <origin xyz="0.005 0.008 -0.020" rpy="0 0 -0.785"/>
         <parent link="r_finger_link"/>
@@ -865,5 +857,5 @@
             <material name="grey"/>
         </visual>
-        <!-- <collision>
+        <collision>
             <origin xyz="-0.05 0 0" rpy="0 0 0"/>
             <geometry>
@@ -871,5 +863,5 @@
                     filename="package://humic_description/meshes/STL/l_shoulder.stl" scale="0.01 0.01 0.01"/>
             </geometry>
-        </collision> -->
+        </collision>
         <inertial>
             <mass value="0.324"/>
@@ -877,8 +869,8 @@
         </inertial>
     </link>
-    <joint name="l_shoulder_joint" type="fixed"> <!-- revolute -->
-        <!-- <axis xyz="0 -1 0" /> -->
-        <!-- <limit velocity="6.5" effort="1000" lower="-3.14" upper="3.14" /> -->
-        <!-- <dynamics damping="0.7"/> -->
+    <joint name="l_shoulder_joint" type="revolute">
+        <axis xyz="0 -1 0" />
+        <limit velocity="6.5" effort="1000" lower="-3.14" upper="3.14" />
+        <dynamics damping="0.7"/>
         <origin xyz="0.004 0.123 0.27" rpy="0 0 0"/>
         <parent link="l_shoulder_link"/>
@@ -894,5 +886,5 @@
             <material name="grey"/>
         </visual>
-        <!-- <collision>
+        <collision>
             <origin xyz="-0.054 -0.125 -0.271" rpy="0 0 0"/>
             <geometry>
@@ -900,5 +892,5 @@
                     filename="package://humic_description/meshes/STL/l_upperArm.stl" scale="0.01 0.01 0.01"/>
             </geometry>
-        </collision> -->
+        </collision>
         <inertial>
             <mass value="0.353"/>
@@ -906,8 +898,8 @@
         </inertial>
     </link>
-    <joint name="l_upperArm_joint" type="fixed"> <!-- revolute -->
-        <!-- <axis xyz="-1 0 0" /> -->
-        <!-- <limit velocity="6.5" effort="1000" lower="-1.57" upper="1.57" /> -->
-        <!-- <dynamics damping="0.7"/> -->
+    <joint name="l_upperArm_joint" type="revolute">
+        <axis xyz="-1 0 0" />
+        <limit velocity="6.5" effort="1000" lower="-1.57" upper="0" />
+        <dynamics damping="0.7"/>
         <origin xyz="0 0.011 0" rpy="0 0 0"/>
         <parent link="l_upperArm_link"/>
@@ -923,5 +915,5 @@
             <material name="grey"/>
         </visual>
-        <!-- <collision>
+        <collision>
             <origin xyz="-0.054 -0.136 -0.271" rpy="0 0 0"/>
             <geometry>
@@ -929,5 +921,5 @@
                     filename="package://humic_description/meshes/STL/l_elbow.stl" scale="0.01 0.01 0.01"/>
             </geometry>
-        </collision> -->
+        </collision>
         <inertial>
             <mass value="0.529"/>
@@ -935,8 +927,8 @@
         </inertial>
     </link>
-    <joint name="l_elbow_joint" type="fixed"> <!-- revolute -->
-        <!-- <axis xyz="-1 0 0" /> -->
-        <!-- <limit velocity="6.5" effort="1000" lower="-1.397" upper="0" /> -->
-        <!-- <dynamics damping="0.7"/> -->
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