Commit message: update urdf scale up

File: humic_description/urdf/humic.urdf.xacro (robot description, xacro)
@@ -1,4 +1,6 @@
 <?xml version="1.0"?>
 <robot name="humic" xmlns:xacro="http://ros.org/wiki/xacro">
+    <!-- some parameters -->
+    <xacro:property name="pi" value="3.141592" />
     <xacro:include filename="$(find humic_description)/urdf/materials.xacro"/>
     <xacro:include filename="$(find humic_description)/urdf/humic.gazebo.xacro"/>
@@ -6,9 +8,9 @@
     <xacro:include filename="$(find humic_description)/urdf/humic.left_transmission.xacro"/>
     <xacro:include filename="$(find humic_description)/urdf/humic.head_transmission.xacro"/>
-    <xacro:include filename="$(find humic_description)/urdf/humic.column_transmission.xacro"/>
+    <!-- <xacro:include filename="$(find humic_description)/urdf/humic.column_transmission.xacro"/> -->
     <!-- base footprint -->
     <link name="base_footprint"/>
     <joint name="base_joint" type="fixed">
-        <origin xyz="0 0 0.035" rpy="0 0 0"/>
+        <origin xyz="0 0 0.0945" rpy="0 0 0"/>
         <parent link="base_footprint"/>
         <child link="base_link"/>
@@ -19,14 +21,14 @@
             <origin xyz="0 0 0" rpy="0 0 0"/>
             <geometry>
-                <mesh filename="package://humic_description/meshes/STL/MobileBody.stl" scale="0.01 0.01 0.01"/>
-            </geometry>
-            <material name="grey"/>
-        </visual>
-        <!-- <collision>
-            <origin xyz="-0.013 0 0.048" rpy="0 0 0"/>
-            <geometry>
-                <mesh filename="package://humic_description/meshes/STL/MobileBody.stl" scale="0.01 0.01 0.01"/>
-            </geometry>
-        </collision> -->
+                <mesh filename="package://humic_description/meshes/STL/MobileBody.stl" scale="0.027 0.027 0.027"/>
+            </geometry>
+            <material name="white"/>
+        </visual>
+        <collision>
+            <origin xyz="0 0 0" rpy="0 0 0"/>
+            <geometry>
+                <mesh filename="package://humic_description/meshes/STL/MobileBody.stl" scale="0.027 0.027 0.027"/>
+            </geometry>
+        </collision>
         <inertial>
             <mass value="64.126"/>
@@ -34,58 +36,58 @@
         </inertial>
     </link>
-    <joint name="front_ultrasound_joint" type="fixed">
-        <origin xyz="0.12 0 0.038" rpy="0 0 0"/>
+    <joint name="front_ultrasonic_joint" type="fixed">
+        <origin xyz="0.335 0 0.102" rpy="0 0 0"/>
         <parent link="base_link"/>
-        <child link="front_ultrasound"/>
-    </joint>
-    <link name="front_ultrasound">
+        <child link="front_ultrasonic"/>
+    </joint>
+    <link name="front_ultrasonic">
         <visual>
             <origin xyz="0 0 0" rpy="0 0 0"/>
             <geometry>
-                <box size="0.002 0.002 0.002"/>
-            </geometry>
-            <material name="red"/>
-        </visual>
-    </link>
-    <joint name="left_ultrasound_joint" type="fixed">
-        <origin xyz="-0.004 0.063 0.038" rpy="0 0 1.57"/>
+                <box size="0.001 0.005 0.005"/>
+            </geometry>
+            <material name="white"/>
+        </visual>
+    </link>
+    <joint name="left_ultrasonic_joint" type="fixed">
+        <origin xyz="-0.01 0.1765 0.102" rpy="0 0 ${pi*0.5}"/>
         <parent link="base_link"/>
-        <child link="left_ultrasound"/>
-    </joint>
-    <link name="left_ultrasound">
+        <child link="left_ultrasonic"/>
+    </joint>
+    <link name="left_ultrasonic">
         <visual>
             <origin xyz="0 0 0" rpy="0 0 0"/>
             <geometry>
-                <box size="0.002 0.002 0.002"/>
-            </geometry>
-            <material name="red"/>
-        </visual>
-    </link>
-    <joint name="right_ultrasound_joint" type="fixed">
-        <origin xyz="-0.004 -0.063 0.038" rpy="0 0 -1.57"/>
+                <box size="0.001 0.005 0.005"/>
+            </geometry>
+            <material name="white"/>
+        </visual>
+    </link>
+    <joint name="right_ultrasonic_joint" type="fixed">
+        <origin xyz="-0.01 -0.1765 0.102" rpy="0 0 ${-pi*0.5}"/>
         <parent link="base_link"/>
-        <child link="right_ultrasound"/>
-    </joint>
-    <link name="right_ultrasound">
+        <child link="right_ultrasonic"/>
+    </joint>
+    <link name="right_ultrasonic">
         <visual>
             <origin xyz="0 0 0" rpy="0 0 0"/>
             <geometry>
-                <box size="0.002 0.002 0.002"/>
-            </geometry>
-            <material name="red"/>
-        </visual>
-    </link>
-    <joint name="rear_ultrasound_joint" type="fixed">
-        <origin xyz="-0.117 0 0.038" rpy="0 0 3.14"/>
+                <box size="0.001 0.005 0.005"/>
+            </geometry>
+            <material name="white"/>
+        </visual>
+    </link>
+    <joint name="rear_ultrasonic_joint" type="fixed">
+        <origin xyz="-0.325 0 0.102" rpy="0 0 ${pi}"/>
         <parent link="base_link"/>
-        <child link="rear_ultrasound"/>
-    </joint>
-    <link name="rear_ultrasound">
+        <child link="rear_ultrasonic"/>
+    </joint>
+    <link name="rear_ultrasonic">
         <visual>
             <origin xyz="0 0 0" rpy="0 0 0"/>
             <geometry>
-                <box size="0.002 0.002 0.002"/>
-            </geometry>
-            <material name="red"/>
+                <box size="0.001 0.005 0.005"/>
+            </geometry>
+            <material name="white"/>
         </visual>
     </link>
@@ -93,7 +95,7 @@
     <!-- front left & rear right couple-->
     <!-- front right & rear left couple-->
-    <joint name="rear_left_wheel_joint" type="continuous">
+    <joint name="rear_left_wheel_joint" type="continuous"> <!-- continuous fixed-->
         <axis xyz="0 -1 0" />
-        <origin xyz="-0.085 0.085 0" rpy="0 0 0"/>
+        <origin xyz="-0.2295 0.2295 0" rpy="0 0 0"/>
         <parent link="base_link"/>
         <child link="rear_left_wheel_link"/>
@@ -104,12 +106,12 @@
             <geometry>
                 <mesh
-                    filename="package://humic_description/meshes/STL/wheel_rear_left.stl" scale="0.01 0.01 0.01"/>
-            </geometry>
-            <material name="white"/>
-        </visual>
-        <collision>
-            <origin xyz="0 0 0" rpy="1.57 0 0"/>
-            <geometry>
-                <cylinder radius="0.04" length="0.037"/>
+                    filename="package://humic_description/meshes/STL/wheel_rear_left.stl" scale="0.027 0.027 0.027"/>
+            </geometry>
+            <material name="white"/>
+        </visual>
+        <collision>
+            <origin xyz="0 0 0" rpy="${pi*0.5} 0 0"/>
+            <geometry>
+                <cylinder radius="0.108" length="0.0999"/>
             </geometry>
         </collision>
@@ -119,7 +121,7 @@
         </inertial>
     </link>
-    <joint name="rear_right_wheel_joint" type="continuous">
+    <joint name="rear_right_wheel_joint" type="continuous"> <!-- continuous fixed -->
         <axis xyz="0 1 0" />
-        <origin xyz="-0.085 -0.085 0" rpy="0 0 0"/>
+        <origin xyz="-0.2295 -0.2295 0" rpy="0 0 0"/>
         <parent link="base_link"/>
         <child link="rear_right_wheel_link"/>
@@ -130,12 +132,12 @@
             <geometry>
                 <mesh
-                    filename="package://humic_description/meshes/STL/wheel_rear_right.stl" scale="0.01 0.01 0.01"/>
-            </geometry>
-            <material name="white"/>
-        </visual>
-        <collision>
-            <origin xyz="0 0 0" rpy="1.57 0 0"/>
-            <geometry>
-                <cylinder radius="0.04" length="0.037"/>
+                    filename="package://humic_description/meshes/STL/wheel_rear_right.stl" scale="0.027 0.027 0.027"/>
+            </geometry>
+            <material name="white"/>
+        </visual>
+        <collision>
+            <origin xyz="0 0 0" rpy="${pi*0.5} 0 0"/>
+            <geometry>
+                <cylinder radius="0.108" length="0.0999"/>
             </geometry>
         </collision>
@@ -145,7 +147,7 @@
         </inertial>
     </link>
-    <joint name="front_right_wheel_joint" type="continuous">
+    <joint name="front_right_wheel_joint" type="continuous"> <!-- continuous fixed -->
         <axis xyz="0 1 0" />
-        <origin xyz="0.085 0.085 0" rpy="0 0 0"/>
+        <origin xyz="0.2295 0.2295 0" rpy="0 0 0"/>
         <parent link="base_link"/>
         <child link="front_right_wheel_link"/>
@@ -156,12 +158,12 @@
             <geometry>
                 <mesh
-                    filename="package://humic_description/meshes/STL/wheel_front_right.stl" scale="0.01 0.01 0.01"/>
-            </geometry>
-            <material name="white"/>
-        </visual>
-        <collision>
-            <origin xyz="0 0 0" rpy="1.57 0 0"/>
-            <geometry>
-                <cylinder radius="0.04" length="0.037"/>
+                    filename="package://humic_description/meshes/STL/wheel_front_right.stl" scale="0.027 0.027 0.027"/>
+            </geometry>
+            <material name="white"/>
+        </visual>
+        <collision>
+            <origin xyz="0 0 0" rpy="${pi*0.5} 0 0"/>
+            <geometry>
+                <cylinder radius="0.108" length="0.0999"/>
             </geometry>
         </collision>
@@ -171,7 +173,7 @@
         </inertial>
     </link>
-    <joint name="front_left_wheel_joint" type="continuous">
+    <joint name="front_left_wheel_joint" type="continuous"> <!-- continuous fixed-->
         <axis xyz="0 -1 0" />
-        <origin xyz="0.085 -0.085 0" rpy="0 0 0"/>
+        <origin xyz="0.2295 -0.2295 0" rpy="0 0 0"/>
         <parent link="base_link"/>
         <child link="front_left_wheel_link"/>
@@ -182,12 +184,12 @@
             <geometry>
                 <mesh
-                    filename="package://humic_description/meshes/STL/wheel_front_left.stl" scale="0.01 0.01 0.01"/>
-            </geometry>
-            <material name="white"/>
-        </visual>
-        <collision>
-            <origin xyz="0 0 0" rpy="1.57 0 0"/>
-            <geometry>
-                <cylinder radius="0.04" length="0.037"/>
+                    filename="package://humic_description/meshes/STL/wheel_front_left.stl" scale="0.027 0.027 0.027"/>
+            </geometry>
+            <material name="white"/>
+        </visual>
+        <collision>
+            <origin xyz="0 0 0" rpy="${pi*0.5} 0 0"/>
+            <geometry>
+                <cylinder radius="0.108" length="0.0999"/>
             </geometry>
         </collision>
@@ -197,5 +199,5 @@
         </inertial>
     </link>
-    <!-- Lift Column -->
+    <!-- Column -->
     <joint name="base_column_joint" type="fixed">
         <origin xyz="0 0 0" rpy="0 0 0"/>
@@ -205,15 +207,15 @@
     <link name="base_column_link">
         <visual>
-            <origin xyz="0.05 0 0.08" rpy="0 0 0"/>
-            <geometry>
-                <mesh
-                    filename="package://humic_description/meshes/STL/column_base.stl" scale="0.01 0.01 0.01"/>
-            </geometry>
-            <material name="white"/>
-        </visual>
-        <collision>
-            <origin xyz="0.05 0 0.15" rpy="0 0 0"/>
-            <geometry>
-                <box size="0.04 0.07 0.105"/>
+            <origin xyz="0.135 0 0.216" rpy="0 0 0"/>
+            <geometry>
+                <mesh
+                    filename="package://humic_description/meshes/STL/column_base.stl" scale="0.027 0.027 0.027"/>
+            </geometry>
+            <material name="white"/>
+        </visual>
+        <collision>
+            <origin xyz="0.135 0 0.405" rpy="0 0 0"/>
+            <geometry>
+                <box size="0.108 0.189 0.2835"/>
             </geometry>
         </collision>
@@ -226,5 +228,5 @@
         <axis xyz="0 0 1" />
         <limit velocity="1" effort="1" lower="0" upper="0.10" />
-        <origin xyz="0.05 0 0.05" rpy="0 0 0"/>
+        <origin xyz="0.135 0 0.135" rpy="0 0 0"/>
         <parent link="base_column_link"/>
         <child link="inner_column_link"/>
@@ -232,8 +234,8 @@
     <link name="inner_column_link">
         <visual>
-            <origin xyz="0 0 0.12" rpy="0 0 0"/>
-            <geometry>
-                <mesh
-                    filename="package://humic_description/meshes/STL/column_inner.stl" scale="0.01 0.01 0.01"/>
+            <origin xyz="0 0 0.324" rpy="0 0 0"/>
+            <geometry>
+                <mesh
+                    filename="package://humic_description/meshes/STL/column_inner.stl" scale="0.027 0.027 0.027"/>
             </geometry>
             <material name="white"/>
@@ -252,15 +254,15 @@
     <link name="torso_link">
         <visual>
-            <origin xyz="-0.016 0 0.275" rpy="0 0 0"/>
-            <geometry>
-                <mesh
-                    filename="package://humic_description/meshes/STL/torso.stl" scale="0.01 0.01 0.01"/>
-            </geometry>
-            <material name="grey"/>
-        </visual>
-        <collision>
-            <origin xyz="-0.003 0 0.23" rpy="0 0 0"/>
-            <geometry>
-                <box size="0.11 0.16 0.15"/>
+            <origin xyz="-0.0432 0 0.7425" rpy="0 0 0"/>
+            <geometry>
+                <mesh
+                    filename="package://humic_description/meshes/STL/torso.stl" scale="0.027 0.027 0.027"/>
+            </geometry>
+            <material name="white"/>
+        </visual>
+        <collision>
+            <origin xyz="-0.0081 0 0.621" rpy="0 0 0"/>
+            <geometry>
+                <box size="0.297 0.432 0.405"/>
             </geometry>
         </collision>
@@ -278,10 +280,10 @@
     <link name="neck_link">
         <visual>
-            <origin xyz="-0.05 0 0" rpy="0 0 0"/>
-            <geometry>
-                <mesh
-                    filename="package://humic_description/meshes/STL/neck.stl" scale="0.01 0.01 0.01"/>
-            </geometry>
-            <material name="grey"/>
+            <origin xyz="-0.135 0 0" rpy="0 0 0"/>
+            <geometry>
+                <mesh
+                    filename="package://humic_description/meshes/STL/neck.stl" scale="0.027 0.027 0.027"/>
+            </geometry>
+            <material name="white"/>
         </visual>
         <inertial>
@@ -292,7 +294,7 @@
     <joint name="neck_joint" type="revolute">
         <axis xyz="0 0 1" />
-        <limit velocity="6.5" effort="1000" lower="-0.7854" upper="0.7854" />
+        <limit velocity="6.5" effort="1000" lower="${-pi*0.5}" upper="${pi*0.5}" />
         <dynamics damping="0.7"/>
-        <origin xyz="0.023 0 0.337" rpy="0 0 0"/>
+        <origin xyz="0.0621 0 0.9099" rpy="0 0 0"/>
         <parent link="neck_link"/>
         <child link="head_link"/>
@@ -300,10 +302,10 @@
     <link name="head_link">
         <visual>
-            <origin xyz="-0.073 0 -0.338" rpy="0 0 0"/>
-            <geometry>
-                <mesh
-                    filename="package://humic_description/meshes/STL/neck_head.stl" scale="0.01 0.01 0.01"/>
-            </geometry>
-            <material name="grey"/>
+            <origin xyz="-0.1971 0 -0.9126" rpy="0 0 0"/>
+            <geometry>
+                <mesh
+                    filename="package://humic_description/meshes/STL/neck_head.stl" scale="0.027 0.027 0.027"/>
+            </geometry>
+            <material name="white"/>
         </visual>
         <inertial>
@@ -314,7 +316,7 @@
     <joint name="head_joint" type="revolute">
         <axis xyz="0 -1 0" />
-        <limit velocity="6.5" effort="1000" lower="-0.7854" upper="0.7854" />
+        <limit velocity="6.5" effort="1000" lower="${-pi*0.5}" upper="${pi*0.5}" />
         <dynamics damping="0.7"/>
-        <origin xyz="0 0 0.02" rpy="0 0.6 0"/>
+        <origin xyz="0 0 0.05" rpy="0 0 0"/>
         <parent link="head_link"/>
         <child link="head_kinect_link"/>
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