Commit message: update URDF

File: humic_description/urdf/humic.urdf.xacro (robot description, xacro)
@@ -8,5 +8,5 @@
     <xacro:include filename="$(find humic_description)/urdf/humic.left_transmission.xacro"/>
     <xacro:include filename="$(find humic_description)/urdf/humic.head_transmission.xacro"/>
-    <!-- <xacro:include filename="$(find humic_description)/urdf/humic.column_transmission.xacro"/> -->
+    <xacro:include filename="$(find humic_description)/urdf/humic.column_transmission.xacro"/>
     <!-- base footprint -->
     <link name="base_footprint"/>
@@ -95,5 +95,5 @@
     <!-- front left & rear right couple-->
     <!-- front right & rear left couple-->
-    <joint name="rear_left_wheel_joint" type="continuous"> <!-- continuous fixed-->
+    <joint name="rear_left_wheel_joint" type="continuous">
         <axis xyz="0 -1 0" />
         <origin xyz="-0.2295 0.2295 0" rpy="0 0 0"/>
@@ -121,5 +121,5 @@
         </inertial>
     </link>
-    <joint name="rear_right_wheel_joint" type="continuous"> <!-- continuous fixed -->
+    <joint name="rear_right_wheel_joint" type="continuous">
         <axis xyz="0 1 0" />
         <origin xyz="-0.2295 -0.2295 0" rpy="0 0 0"/>
@@ -147,5 +147,5 @@
         </inertial>
     </link>
-    <joint name="front_right_wheel_joint" type="continuous"> <!-- continuous fixed -->
+    <joint name="front_right_wheel_joint" type="continuous">
         <axis xyz="0 1 0" />
         <origin xyz="0.2295 0.2295 0" rpy="0 0 0"/>
@@ -173,5 +173,5 @@
         </inertial>
     </link>
-    <joint name="front_left_wheel_joint" type="continuous"> <!-- continuous fixed-->
+    <joint name="front_left_wheel_joint" type="continuous">
         <axis xyz="0 -1 0" />
         <origin xyz="0.2295 -0.2295 0" rpy="0 0 0"/>
@@ -207,5 +207,5 @@
     <link name="base_column_link">
         <visual>
-            <origin xyz="0.135 0 0.216" rpy="0 0 0"/>
+            <origin xyz="0.135 0 0.2" rpy="0 0 0"/>
             <geometry>
                 <mesh
@@ -215,7 +215,8 @@
         </visual>
         <collision>
-            <origin xyz="0.135 0 0.405" rpy="0 0 0"/>
-            <geometry>
-                <box size="0.108 0.189 0.2835"/>
+            <origin xyz="0.135 0 0.2" rpy="0 0 0"/>
+            <geometry>
+                <mesh
+                    filename="package://humic_description/meshes/STL/column_base.stl" scale="0.027 0.027 0.027"/>
             </geometry>
         </collision>
@@ -227,6 +228,6 @@
     <joint name="inner_column_joint" type="prismatic">
         <axis xyz="0 0 1" />
-        <limit velocity="1" effort="1" lower="0" upper="0.10" />
-        <origin xyz="0.135 0 0.135" rpy="0 0 0"/>
+        <limit velocity="0.01" effort="1000" lower="0" upper="0.20" />
+        <origin xyz="0.135 0 0.1" rpy="0 0 0"/>
         <parent link="base_column_link"/>
         <child link="inner_column_link"/>
@@ -234,5 +235,5 @@
     <link name="inner_column_link">
         <visual>
-            <origin xyz="0 0 0.324" rpy="0 0 0"/>
+            <origin xyz="0 0 0.3" rpy="0 0 0"/>
             <geometry>
                 <mesh
@@ -241,4 +242,11 @@
             <material name="white"/>
         </visual>
+        <collision>
+            <origin xyz="0 0 0.3" rpy="0 0 0"/>
+            <geometry>
+                <mesh
+                    filename="package://humic_description/meshes/STL/column_inner.stl" scale="0.027 0.027 0.027"/>
+            </geometry>
+        </collision>
         <inertial>
             <mass value="2.349"/>
@@ -318,5 +326,5 @@
         <limit velocity="6.5" effort="1000" lower="${-pi*0.5}" upper="${pi*0.5}" />
         <dynamics damping="0.7"/>
-        <origin xyz="0 0 0.05" rpy="0 0 0"/>
+        <origin xyz="0 0 0.05" rpy="0 0.6 0"/>
         <parent link="head_link"/>
         <child link="head_kinect_link"/>
@@ -586,6 +594,6 @@
     <joint name="r_finger1_1_joint" type="revolute">
         <axis xyz="1 0 0" />
-        <limit velocity="1" effort="1" lower="0" upper="${pi*0.5}" />
-        <dynamics damping="0.2"/>
+        <limit velocity="10" effort="1000" lower="0" upper="${pi*0.5}" />
+        <dynamics damping="0.7"/>
         <origin xyz="0.0324 -0.0162 -0.0972" rpy="0 0 0"/>
         <parent link="r_finger_link"/>
@@ -615,6 +623,6 @@
     <joint name="r_finger1_2_joint" type="revolute">
         <axis xyz="1 0 0" />
-        <limit velocity="1" effort="1" lower="0" upper="${pi*0.5}" />
-        <dynamics damping="0.2"/>
+        <limit velocity="10" effort="1000" lower="0" upper="${pi*0.5}" />
+        <dynamics damping="0.7"/>
         <origin xyz="0 0 -0.054" rpy="0 0 0"/>
         <parent link="r_finger1_1_link"/>
@@ -644,6 +652,6 @@
     <joint name="r_finger2_1_joint" type="revolute">
         <axis xyz="1 0 0" />
-        <limit velocity="1" effort="1" lower="0" upper="${pi*0.5}" />
-        <dynamics damping="0.2"/>
+        <limit velocity="10" effort="1000" lower="0" upper="${pi*0.5}" />
+        <dynamics damping="0.7"/>
         <origin xyz="0.0108 -0.0162 -0.0972" rpy="0 0 0"/>
         <parent link="r_finger_link"/>
@@ -673,6 +681,6 @@
     <joint name="r_finger2_2_joint" type="revolute">
         <axis xyz="1 0 0" />
-        <limit velocity="1" effort="1" lower="0" upper="${pi*0.5}" />
-        <dynamics damping="0.2"/>
+        <limit velocity="10" effort="1000" lower="0" upper="${pi*0.5}" />
+        <dynamics damping="0.7"/>
         <origin xyz="0 0 -0.0567" rpy="0 0 0"/>
         <parent link="r_finger2_1_link"/>
@@ -702,6 +710,6 @@
     <joint name="r_finger3_1_joint" type="revolute">
         <axis xyz="1 0 0" />
-        <limit velocity="1" effort="1" lower="0" upper="${pi*0.5}" />
-        <dynamics damping="0.2"/>
+        <limit velocity="10" effort="1000" lower="0" upper="${pi*0.5}" />
+        <dynamics damping="0.7"/>
         <origin xyz="-0.0108 -0.0162 -0.0972" rpy="0 0 0"/>
         <parent link="r_finger_link"/>
@@ -731,6 +739,6 @@
     <joint name="r_finger3_2_joint" type="revolute">
         <axis xyz="1 0 0" />
-        <limit velocity="1" effort="1" lower="0" upper="${pi*0.5}" />
-        <dynamics damping="0.2"/>
+        <limit velocity="10" effort="1000" lower="0" upper="${pi*0.5}" />
+        <dynamics damping="0.7"/>
         <origin xyz="0 0 -0.0459" rpy="0 0 0"/>
         <parent link="r_finger3_1_link"/>
@@ -760,6 +768,6 @@
     <joint name="r_finger4_1_joint" type="revolute">
         <axis xyz="1 0 0" />
-        <limit velocity="1" effort="1" lower="0" upper="${pi*0.5}" />
-        <dynamics damping="0.2"/>
+        <limit velocity="10" effort="1000" lower="0" upper="${pi*0.5}" />
+        <dynamics damping="0.7"/>
         <origin xyz="-0.0324 -0.0162 -0.0972" rpy="0 0 0"/>
         <parent link="r_finger_link"/>
@@ -789,6 +797,6 @@
     <joint name="r_finger4_2_joint" type="revolute">
         <axis xyz="1 0 0" />
-        <limit velocity="1" effort="1" lower="0" upper="${pi*0.5}" />
-        <dynamics damping="0.2"/>
+        <limit velocity="10" effort="1000" lower="0" upper="${pi*0.5}" />
+        <dynamics damping="0.7"/>
         <origin xyz="0 0 -0.0405" rpy="0 0 0"/>
         <parent link="r_finger4_1_link"/>
@@ -818,6 +826,6 @@
     <joint name="r_thumb_joint" type="revolute">
         <axis xyz="0 0 1" />
-        <limit velocity="1" effort="1" lower="0" upper="${pi*0.25}" />
-        <dynamics damping="0.2"/>
+        <limit velocity="10" effort="1000" lower="0" upper="${pi*0.25}" />
+        <dynamics damping="0.7"/>
         <origin xyz="0.0135 0.0216 -0.054" rpy="0 0 ${-pi*0.25}"/>
         <parent link="r_finger_link"/>
@@ -1058,6 +1066,6 @@
     <joint name="l_finger1_1_joint" type="revolute">
         <axis xyz="-1 0 0" />
-        <limit velocity="1" effort="1" lower="0" upper="${pi*0.5}" />
-        <dynamics damping="0.2"/>
+        <limit velocity="10" effort="1000" lower="0" upper="${pi*0.5}" />
+        <dynamics damping="0.7"/>
         <origin xyz="0.0324 0.0162 -0.0972" rpy="0 0 0"/>
         <parent link="l_finger_link"/>
@@ -1087,6 +1095,6 @@
     <joint name="l_finger1_2_joint" type="revolute">
         <axis xyz="-1 0 0" />
-        <limit velocity="1" effort="1" lower="0" upper="${pi*0.5}" />
-        <dynamics damping="0.2"/>
+        <limit velocity="10" effort="1000" lower="0" upper="${pi*0.5}" />
+        <dynamics damping="0.7"/>
         <origin xyz="0 0 -0.054" rpy="0 0 0"/>
         <parent link="l_finger1_1_link"/>
@@ -1116,6 +1124,6 @@
     <joint name="l_finger2_1_joint" type="revolute">
         <axis xyz="-1 0 0" />
-        <limit velocity="1" effort="1" lower="0" upper="${pi*0.5}" />
-        <dynamics damping="0.2"/>
+        <limit velocity="10" effort="1000" lower="0" upper="${pi*0.5}" />
+        <dynamics damping="0.7"/>
         <origin xyz="0.0108 0.0162 -0.0972" rpy="0 0 0"/>
         <parent link="l_finger_link"/>
@@ -1145,6 +1153,6 @@
     <joint name="l_finger2_2_joint" type="revolute">
         <axis xyz="-1 0 0" />
-        <limit velocity="1" effort="1" lower="0" upper="${pi*0.5}" />
-        <dynamics damping="0.2"/>
+        <limit velocity="10" effort="1000" lower="0" upper="${pi*0.5}" />
+        <dynamics damping="0.7"/>
         <origin xyz="0 0 -0.0567" rpy="0 0 0"/>
         <parent link="l_finger2_1_link"/>
@@ -1174,6 +1182,6 @@
     <joint name="l_finger3_1_joint" type="revolute">
         <axis xyz="-1 0 0" />
-        <limit velocity="1" effort="1" lower="0" upper="${pi*0.5}" />
-        <dynamics damping="0.2"/>
+        <limit velocity="10" effort="1000" lower="0" upper="${pi*0.5}" />
+        <dynamics damping="0.7"/>
         <origin xyz="-0.0108 0.0162 -0.0972" rpy="0 0 0"/>
         <parent link="l_finger_link"/>
@@ -1203,6 +1211,6 @@
     <joint name="l_finger3_2_joint" type="revolute">
         <axis xyz="-1 0 0" />
-        <limit velocity="1" effort="1" lower="0" upper="${pi*0.5}" />
-        <dynamics damping="0.2"/>
+        <limit velocity="10" effort="1000" lower="0" upper="${pi*0.5}" />
+        <dynamics damping="0.7"/>
         <origin xyz="0 0 -0.0459" rpy="0 0 0"/>
         <parent link="l_finger3_1_link"/>
@@ -1232,6 +1240,6 @@
     <joint name="l_finger4_1_joint" type="revolute">
         <axis xyz="-1 0 0" />
-        <limit velocity="1" effort="1" lower="0" upper="${pi*0.5}" />
-        <dynamics damping="0.2"/>
+        <limit velocity="10" effort="1000" lower="0" upper="${pi*0.5}" />
+        <dynamics damping="0.7"/>
         <origin xyz="-0.0324 0.0162 -0.0972" rpy="0 0 0"/>
         <parent link="l_finger_link"/>
@@ -1261,6 +1269,6 @@
     <joint name="l_finger4_2_joint" type="revolute">
         <axis xyz="-1 0 0" />
-        <limit velocity="1" effort="1" lower="0" upper="${pi*0.5}" />
-        <dynamics damping="0.2"/>
+        <limit velocity="10" effort="1000" lower="0" upper="${pi*0.5}" />
+        <dynamics damping="0.7"/>
         <origin xyz="0 0 -0.0405" rpy="0 0 0"/>
         <parent link="l_finger4_1_link"/>
@@ -1290,6 +1298,6 @@
     <joint name="l_thumb_joint" type="revolute">
         <axis xyz="0 0 -1" />
-        <limit velocity="1" effort="1" lower="0" upper="${pi*0.25}" />
-        <dynamics damping="0.2"/>
+        <limit velocity="10" effort="1000" lower="0" upper="${pi*0.25}" />
+        <dynamics damping="0.7"/>
         <origin xyz="0.0135 -0.0216 -0.054" rpy="0 0 ${pi*0.25}"/>
         <parent link="l_finger_link"/>

Commit message: update 2021 05 05

File: humic_description/urdf/humic.urdf.xacro (robot description, xacro)
@@ -594,5 +594,5 @@
     <joint name="r_finger1_1_joint" type="revolute">
         <axis xyz="1 0 0" />
-        <limit velocity="10" effort="1000" lower="0" upper="${pi*0.5}" />
+        <limit velocity="3" effort="1000" lower="0" upper="${pi*0.5}" />
         <dynamics damping="0.7"/>
         <origin xyz="0.0324 -0.0162 -0.0972" rpy="0 0 0"/>
@@ -623,5 +623,5 @@
     <joint name="r_finger1_2_joint" type="revolute">
         <axis xyz="1 0 0" />
-        <limit velocity="10" effort="1000" lower="0" upper="${pi*0.5}" />
+        <limit velocity="3" effort="1000" lower="0" upper="${pi*0.5}" />
         <dynamics damping="0.7"/>
         <origin xyz="0 0 -0.054" rpy="0 0 0"/>
@@ -652,5 +652,5 @@
     <joint name="r_finger2_1_joint" type="revolute">
         <axis xyz="1 0 0" />
-        <limit velocity="10" effort="1000" lower="0" upper="${pi*0.5}" />
+        <limit velocity="3" effort="1000" lower="0" upper="${pi*0.5}" />
         <dynamics damping="0.7"/>
         <origin xyz="0.0108 -0.0162 -0.0972" rpy="0 0 0"/>
@@ -681,5 +681,5 @@
     <joint name="r_finger2_2_joint" type="revolute">
         <axis xyz="1 0 0" />
-        <limit velocity="10" effort="1000" lower="0" upper="${pi*0.5}" />
+        <limit velocity="3" effort="1000" lower="0" upper="${pi*0.5}" />
         <dynamics damping="0.7"/>
         <origin xyz="0 0 -0.0567" rpy="0 0 0"/>
@@ -710,5 +710,5 @@
     <joint name="r_finger3_1_joint" type="revolute">
         <axis xyz="1 0 0" />
-        <limit velocity="10" effort="1000" lower="0" upper="${pi*0.5}" />
+        <limit velocity="3" effort="1000" lower="0" upper="${pi*0.5}" />
         <dynamics damping="0.7"/>
         <origin xyz="-0.0108 -0.0162 -0.0972" rpy="0 0 0"/>
@@ -739,5 +739,5 @@
     <joint name="r_finger3_2_joint" type="revolute">
         <axis xyz="1 0 0" />
-        <limit velocity="10" effort="1000" lower="0" upper="${pi*0.5}" />
+        <limit velocity="3" effort="1000" lower="0" upper="${pi*0.5}" />
         <dynamics damping="0.7"/>
         <origin xyz="0 0 -0.0459" rpy="0 0 0"/>
@@ -768,5 +768,5 @@
     <joint name="r_finger4_1_joint" type="revolute">
         <axis xyz="1 0 0" />
-        <limit velocity="10" effort="1000" lower="0" upper="${pi*0.5}" />
+        <limit velocity="3" effort="1000" lower="0" upper="${pi*0.5}" />
         <dynamics damping="0.7"/>
         <origin xyz="-0.0324 -0.0162 -0.0972" rpy="0 0 0"/>
@@ -797,5 +797,5 @@
     <joint name="r_finger4_2_joint" type="revolute">
         <axis xyz="1 0 0" />
-        <limit velocity="10" effort="1000" lower="0" upper="${pi*0.5}" />
+        <limit velocity="3" effort="1000" lower="0" upper="${pi*0.5}" />
         <dynamics damping="0.7"/>
         <origin xyz="0 0 -0.0405" rpy="0 0 0"/>
@@ -826,5 +826,5 @@
     <joint name="r_thumb_joint" type="revolute">
         <axis xyz="0 0 1" />
-        <limit velocity="10" effort="1000" lower="0" upper="${pi*0.25}" />
+        <limit velocity="3" effort="1000" lower="0" upper="${pi*0.25}" />
         <dynamics damping="0.7"/>
         <origin xyz="0.0135 0.0216 -0.054" rpy="0 0 ${-pi*0.25}"/>

Commit message: modify 2020 05 18

File: humic_description/urdf/humic.urdf.xacro (robot description, xacro)
@@ -228,6 +228,8 @@
     <joint name="inner_column_joint" type="prismatic">
         <axis xyz="0 0 1" />
-        <limit velocity="0.01" effort="1000" lower="0" upper="0.20" />
-        <origin xyz="0.135 0 0.1" rpy="0 0 0"/>
+        <limit velocity="0.01" effor="1000" lower="0" upper="0.20" />
+        <origin xyz="0.135 0 0.3" rpy="0 0 0"/>
+        <!-- <limit velocity="0.01" effort="1000" lower="0" upper="0.5" /> -->
+        <!-- <origin xyz="0.135 0 0.05" rpy="0 0 0"/> -->
         <parent link="base_column_link"/>
         <child link="inner_column_link"/>
@@ -235,5 +237,5 @@
     <link name="inner_column_link">
         <visual>
-            <origin xyz="0 0 0.3" rpy="0 0 0"/>
+            <origin xyz="0 0 0.4" rpy="0 0 0"/>
             <geometry>
                 <mesh
@@ -243,5 +245,5 @@
         </visual>
         <collision>
-            <origin xyz="0 0 0.3" rpy="0 0 0"/>
+            <origin xyz="0 0 0.4" rpy="0 0 0"/>
             <geometry>
                 <mesh
@@ -262,5 +264,5 @@
     <link name="torso_link">
         <visual>
-            <origin xyz="-0.0432 0 0.7425" rpy="0 0 0"/>
+            <origin xyz="-0.0432 0 0.675" rpy="0 0 0"/>
             <geometry>
                 <mesh
@@ -282,5 +284,5 @@
     <!-- head(Pan(neck), Tile(head), Kinect V2)-->
     <joint name="torso_neck_joint" type="fixed">
-        <origin xyz="0 0 0" rpy="0 0 0"/>
+        <origin xyz="0 0 -0.0675" rpy="0 0 0"/>
         <parent link="torso_link"/>
         <child link="neck_link"/>
@@ -326,5 +328,5 @@
         <limit velocity="6.5" effort="1000" lower="${-pi*0.5}" upper="${pi*0.5}" />
         <dynamics damping="0.7"/>
-        <origin xyz="0 0 0.05" rpy="0 0.6 0"/>
+        <origin xyz="0 0 0.05" rpy="0 0 0"/>
         <parent link="head_link"/>
         <child link="head_kinect_link"/>
@@ -373,5 +375,5 @@
     <link name="imu_link">
         <visual>
-            <origin xyz="0.0621 0.0216 0.729" rpy="0 0 0"/>
+            <origin xyz="0.0621 0.0216 0.6615" rpy="0 0 0"/>
             <geometry>
                 <box size="0.00135 0.0054 0.0054"/>
@@ -382,5 +384,5 @@
     <!-- Right ARM -->
     <joint name="r_arm_body_joint" type="fixed">
-        <origin xyz="0 0 0" rpy="0 0 0"/>
+        <origin xyz="0 0 -0.0675" rpy="0 0 0"/>
         <parent link="torso_link"/>
         <child link="r_shoulder_link"/>
@@ -855,4 +857,5 @@
     <!-- Left ARM -->
     <joint name="l_arm_body_joint" type="fixed">
+        <origin xyz="0 0 -0.0675" rpy="0 0 0"/>
         <parent link="torso_link"/>
         <child link="l_shoulder_link"/>

Commit message: Update humic.urdf.xacro

File: humic_description/urdf/humic.urdf.xacro (robot description, xacro)
@@ -230,5 +230,5 @@
         <limit velocity="0.01" effor="1000" lower="0" upper="0.20" />
         <origin xyz="0.135 0 0.3" rpy="0 0 0"/>
-        <!-- <limit velocity="0.01" effort="1000" lower="0" upper="0.5" /> -->
+        <!-- <limit velocity="0.01" effort="1000" lower="0" upper="0.45" /> -->
         <!-- <origin xyz="0.135 0 0.05" rpy="0 0 0"/> -->
         <parent link="base_column_link"/>

Commit message: update 2021 05 20

File: humic_description/urdf/humic.urdf.xacro (robot description, xacro)
@@ -228,8 +228,6 @@
     <joint name="inner_column_joint" type="prismatic">
         <axis xyz="0 0 1" />
-        <limit velocity="0.01" effor="1000" lower="0" upper="0.20" />
-        <origin xyz="0.135 0 0.3" rpy="0 0 0"/>
-        <!-- <limit velocity="0.01" effort="1000" lower="0" upper="0.45" /> -->
-        <!-- <origin xyz="0.135 0 0.05" rpy="0 0 0"/> -->
+        <limit velocity="0.01" effor="1000" lower="0" upper="0.50" />
+        <origin xyz="0.135 0 0.05" rpy="0 0 0"/>
         <parent link="base_column_link"/>
         <child link="inner_column_link"/>

Commit message: Update humic.urdf.xacro

File: humic_description/urdf/humic.urdf.xacro (robot description, xacro)
@@ -270,5 +270,5 @@
         </visual>
         <collision>
-            <origin xyz="-0.0081 0 0.621" rpy="0 0 0"/>
+            <origin xyz="-0.0081 0 0.55" rpy="0 0 0"/>
             <geometry>
                 <box size="0.297 0.432 0.405"/>

Commit message: Update humic.urdf.xacro

File: humic_description/urdf/humic.urdf.xacro (robot description, xacro)
@@ -881,5 +881,5 @@
     </link>
     <joint name="l_shoulder_joint" type="revolute">
-        <axis xyz="0 -1 0" />
+        <axis xyz="0 1 0" />
         <limit velocity="6.5" effort="1000" lower="${-pi}" upper="${pi}" />
         <dynamics damping="0.7"/>
@@ -968,5 +968,5 @@
     </link>
     <joint name="l_foreArm_joint" type="revolute">
-        <axis xyz="0 0 1" />
+        <axis xyz="0 0 -1" />
         <limit velocity="6.5" effort="1000" lower="${-pi}" upper="${pi}" />
         <dynamics damping="0.7"/>
@@ -1026,5 +1026,5 @@
     </link>
     <joint name="l_wrist_joint" type="revolute">
-        <axis xyz="0 0 1" />
+        <axis xyz="0 0 -1" />
         <limit velocity="13" effort="1000" lower="${-pi}" upper="${pi}" />
         <dynamics damping="0.7"/>
